File: ADS1299-test_circuit.sch (KiCad schematic (older format))
At the start: 109 parts, among them J1 OUT, J2 GND, J3 GND, P1 +5V, P10 IN2, P11 IN6, P12 IN5, P13 IN1, P14 BiasOut_C, P15 BiasOut_R, P16 BiasIn_C, P17 BiasIn_R, P18 Temp5030, P19 Daisy, P2 Temp5025, P20 Sw_pwdn, P21 Electrodes, P22 D/Ref, P23 -5V, P3 +3.3V, P4 +2.5V, P5 -2.5V, P6 IN4, P7 IN8, P8 IN3, P9 IN7, U1 REF5025, U2 REF5030, U3 ADS1299, U4 OPA735

Commit message: Arreglos LCI
- Pistas mas gruesas donde es posible.
- Pines de TEMP se corrigieron a 2.57mm.
Parts:
- P18, P2: footprint Pin_Headers:Pin_Header_Straight_1x01_Pitch1.27mm -> Pin_Headers:Pin_Header_Straight_1x01_Pitch2.54mm
Changed lines of the file:
@@
 F 0 "P2" H 2300 950 50  0000 C CNN
 F 1 "Temp5025" V 2400 850 50  0000 C CNN
-F 2 "Pin_Headers:Pin_Header_Straight_1x01_Pitch1.27mm" H 2300 850 50  0001 C CNN
+F 2 "Pin_Headers:Pin_Header_Straight_1x01_Pitch2.54mm" H 2300 850 50  0001 C CNN
 F 3 "" H 2300 850 50  0000 C CNN
 	1    2300 850
@@
 F 0 "P18" H 7600 950 50  0000 C CNN
 F 1 "Temp5030" V 7700 850 50  0000 C CNN
-F 2 "Pin_Headers:Pin_Header_Straight_1x01_Pitch1.27mm" H 7600 850 50  0001 C CNN
+F 2 "Pin_Headers:Pin_Header_Straight_1x01_Pitch2.54mm" H 7600 850 50  0001 C CNN
 F 3 "" H 7600 850 50  0000 C CNN
 	1    7600 850

Commit message: Correcciones LCI
Ahora las vias son pines con thermal relief.
Parts:
- added J10, J11, J12, J13, J14, J15, J16, J17, J18, J19, J20, J21, J22, J23, J24, J25, J26, J27, J28, J29, J30, J31, J32, J33, J4, J5, J6, J7, J8, J9: CONN_01X01, Pin_Headers:Pin_Header_Straight_1x01_Pitch2.54mm, symbol CONN_01X01
Connections:
- net GND: now also J10.1 (P1), J11.1 (P1), J12.1 (P1), J13.1 (P1), J14.1 (P1), J15.1 (P1), J16.1 (P1), J17.1 (P1), J18.1 (P1), J19.1 (P1), J20.1 (P1), J21.1 (P1), J22.1 (P1), J23.1 (P1), J24.1 (P1), J25.1 (P1), J26.1 (P1), J27.1 (P1), J28.1 (P1), J29.1 (P1), J30.1 (P1), J31.1 (P1), J32.1 (P1), J33.1 (P1), J4.1 (P1), J5.1 (P1), J6.1 (P1), J7.1 (P1), J8.1 (P1), J9.1 (P1)
Other:
- note added: "VIAS"
- moved on the sheet: J2, J3, P21
